File: CPC stuff/ramcard/ramcard.sch (KiCad schematic (older format))
At the start: 44 parts

Commit message: * Blinkdel for attiny2313 (and easier to adapt)  * Ramcard schematic update
git-svn-id: svn://pulkomandy.tk/avrstuff@36 c6672c3c-f6b6-47f9-9001-1fd6b12fecbe
Parts:
- C?: value CP1 -> 1µF
- D?: value DIODE -> BZX55C
- D?: value DIODE -> 1N4148
- R?: value R -> 1K
- R?: value R -> 10K
Connections:
- wire segments 105 -> 117
Other:
- moved on the sheet: BT?, C?, D?, Q?, R?

Commit message: Début de reproduction du routage. Quelques ajouts et corrections dans le schéma.
git-svn-id: svn://pulkomandy.tk/avrstuff@37 c6672c3c-f6b6-47f9-9001-1fd6b12fecbe
Parts:
- BT1: renamed from BT?; value BATTERY -> CR2032
- D12: renamed from D?; value DIODE -> BAT85
- gave numbers to parts that had none: 35
- renumbered SW_CFG to SW_CFG1, SW_ROMEN to SW_ROMEN1
Connections:
- net labels added: +BATT, A10, A11, A12, A13, A14, A15, A16, A18, A8, A9, AC0, AC1, AC2, AC3, AC4, D0, D1, D2, D3, D4, D5, D6, D7, I1, I2, I3, I4, IS0, IS1, IS2
- net labels removed: A[0..3], A[4..7], CPC_A13, CPC_A14, CPC_A15
- wire segments 117 -> 193
Other:
- moved on the sheet: BT1, C2, C5, D11, D12, R10, R2, R3, R4, R5, R6, SW_CFG1

Commit message: Routing finished. Schematic is now 100% identical to the original.
git-svn-id: svn://pulkomandy.tk/avrstuff@38 c6672c3c-f6b6-47f9-9001-1fd6b12fecbe
Parts:
- added unit 3 of U1
Connections:
- net labels removed: A16, A18
- wire segments 193 -> 207
- no-connect marks 13 -> 27
Other:
- moved on the sheet: BT1, C1, C2, C3, C4, C5, D1, D11, D12, D2, Q1, R1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
