File: CPC stuff/cpc_serial_2313/cpcser.sch (KiCad schematic (older format))
At the start: 25 parts, among them J1 DB9, P1 CONN_25X2, P2 FWUP, U2 ATTINY2313MLF, U3 MAX232, U4 74LS02, X1 CRYSTAL

Commit message: * Fix schematic for µSerial : add "local handshake" to make some PCs happy  * Some improvements to the test code.
git-svn-id: svn://pulkomandy.tk/avrstuff@42 c6672c3c-f6b6-47f9-9001-1fd6b12fecbe
Connections:
- net at J1.1: now also J1.4, J1.6 (P6)
- net at J1.7 (P7): now also J1.8 (P8)
Changed lines of the file:
@@
-EESchema Schematic File Version 2  date 07/11/2010 23:45:51
+EESchema Schematic File Version 2  date 14/05/2011 19:38:41
 LIBS:power
 LIBS:device
@@
 LIBS:attiny
 LIBS:cpcser-cache
-EELAYER 24  0
+EELAYER 25  0
 EELAYER END
 $Descr User 8000 7500
+encoding utf-8
 Sheet 1 1
 Title "Micro-serial RS232 interface for CPC"
-Date "7 nov 2010"
+Date "14 may 2011"
 Rev "0.2"
 Comp "Shinra/PulkoTronics"
@@
 $EndDescr
 Wire Wire Line
+	1150 4800 1200 4800
+Wire Wire Line
+	1200 4800 1200 5000
+Wire Wire Line
+	1200 5000 1150 5000
+Wire Wire Line
 	1150 5300 1150 5350
 Wire Wire Line
@@
 Wire Wire Line
 	2500 3900 2500 4650
+Wire Wire Line
+	1150 4500 1150 4600
+Wire Wire Line
+	1150 4600 1400 4600
+Wire Wire Line
+	1400 4600 1400 4950
+Wire Wire Line
+	1400 4950 1250 4950
+Wire Wire Line
+	1250 4950 1250 5100
+Wire Wire Line
+	1250 5100 1150 5100
 $Comp
 L GND #PWR01
