File: CPC stuff/gordon/ramcard.sch (KiCad schematic (older format))
At the start: 39 parts, among them P1 CONN_25X2, Q1 BC307, U1 74LS00, U2 74LS138, U3 74LS32, U4 74LS374, U5 74LS85, U6 SRAM_512KO

Commit message: fix wire-or (backward diodes) and improve routing. 15 straps left...
git-svn-id: svn://pulkomandy.tk/avrstuff@41 c6672c3c-f6b6-47f9-9001-1fd6b12fecbe
Parts:
- removed BT1: CR2032, symbol BATTERY
- removed C1: 1µF, symbol CP1
- removed D12: BAT85, symbol DIODE
- removed Q1: BC307, symbol BC307
- removed R1: 10K, symbol R
- removed R10: R, symbol R
- removed R3, R4, R5, R6: 10KR, symbol R
- removed R7: 1K, symbol R
- removed SW_CFG1: DIPS_08, symbol DIPS_08
- removed U5: 74LS85, symbol 74LS85
- added JP1: JUMPER, symbol JUMPER
- D1: value 1N4148 -> DIODE
- D2: value BZX55C -> DIODE
Connections:
- net labels added: ACFG, AX17, AX18, CE
- net labels removed: AC2, AC3, AC4, I1, I2, I3, I4, WRITE_EN
- wire segments 207 -> 166
- no-connect marks 27 -> 19
Other:
- note removed: "To address comparator"
- note removed: "To individual rom select"
- moved on the sheet: C2, C3, C4, C5, R2, R9, U1A, U1C, U1D, U3A, U3D

Commit message: Lots of fixes to Gordon after tests on the first prototype.
git-svn-id: svn://pulkomandy.tk/avrstuff@43 c6672c3c-f6b6-47f9-9001-1fd6b12fecbe
Parts:
- removed JP1: JUMPER, symbol JUMPER
- removed R9: R, symbol R
- removed unit 2 of U3
- added K1: CONN_3, symbol CONN_3
Connections:
- net labels added: RD
- net labels removed: +BATT, WRITE
- wire segments 166 -> 161
- no-connect marks 19 -> 18
Other:
- note removed: "Write detection"
- moved on the sheet: C2, C3, C4, C5, D13, U1A, U1B, U1D, U3A, U3C, U3D

Commit message: Replace broken GORDON schematics with reverse engineering of MegaFLASH one, to serve as a base for improvements.
git-svn-id: svn://pulkomandy.tk/avrstuff@70 c6672c3c-f6b6-47f9-9001-1fd6b12fecbe
Parts:
- removed D1, D10, D3, D4, D5, D6, D7, D8, D9: DIODE, symbol DIODE
- removed K1: CONN_3, symbol CONN_3
- removed R8: R, symbol R
- removed SW_ROMEN1: DIPS_08, symbol DIPS_08
- removed U1: 74LS00, symbol 74LS00
- removed U2: 74LS138, symbol 74LS138
- removed U4: 74LS374, symbol 74LS374
- removed U6: SRAM_512KO, symbol SRAM_512KO
- added D?: LED, symbol LED
- added R? (x2): 1KR, symbol R
- added R?: 220R, symbol R
- added SW? (x2): SWITCH_INV, symbol SWITCH_INV
- added U1: 74LS574, symbol 74LS574
- added unit 2 of U2
- added U3: 74LS32, symbol 74LS32
- added U4: 74LS02, symbol 74LS02
- added U5: 74LS20, symbol 74LS20
- added U6: 29C040, symbol 29C040
- R2: value 10KR -> 1KR
- renumbered U3 to U2
Connections:
- net labels added: /CE, /WE, Q0, Q1, Q2, Q3, Q4, Q5, Q6, Q7, R0EN, R7EN, RDWR, ROMACC
- net labels removed: AC0, AC1, ACFG, AX17, AX18, IS0, IS1, IS2, MATCH, ROM_ACC, ROM_ACTIVE, _A3
- wire segments 161 -> 131
Other:
- note added: "DSDP\nSWITCH"
- note removed: "Individual ROM selection"
- note removed: "Rom access detection"
- note removed: "demultiplexer"
- moved on the sheet: C2, C3, C4, C5, D11, D13, D2, P1, R2

Commit message: * Finished schematic (now a clearer version of the MegaFlash one)  * Started a first try at routing.
git-svn-id: svn://pulkomandy.tk/avrstuff@71 c6672c3c-f6b6-47f9-9001-1fd6b12fecbe
Parts:
- added SW1: SWITCH_DSDP, symbol SWITCH_DSDP
- gave numbers to parts that had none: 6
Connections:
- wire segments 131 -> 132
Other:
- note removed: "DSDP\nSWITCH"
