File: CPC stuff/gordon/ramcard.sch (KiCad schematic (older format))
At the start: 22 parts, among them P1 CONN_25X2, SW1 SWITCH_DSDP, SW2 SWITCH_INV, SW3 SWITCH_INV, U1 74LS574, U2 74LS32, U3 74LS32, U4 74LS02, U5 74LS20, U6 29C040

Commit message: Routing done added reset button and ALL ROMS OFF mode (remove JP0)
git-svn-id: svn://pulkomandy.tk/avrstuff@74 c6672c3c-f6b6-47f9-9001-1fd6b12fecbe
Parts:
- added R5: 10KR, symbol R
- added SW4: SW_PUSH, symbol SW_PUSH
- SW1: value SWITCH_DSDP -> WRITE
- SW2: value SWITCH_INV -> ROM7
- SW3: value SWITCH_INV -> ROM0
Connections:
- net labels added: BUSRESET
- wire segments 132 -> 134
- no-connect marks 18 -> 17
Changed lines of the file:
@@
-EESchema Schematic File Version 2  date 22/09/2012 18:26:40
+EESchema Schematic File Version 2  date 29/09/2012 15:56:12
 LIBS:device
 LIBS:power
@@
 Sheet 1 1
 Title "Ramcard"
-Date "22 sep 2012"
+Date "29 sep 2012"
 Rev ""
 Comp "Ram7"
@@
 Comment4 ""
 $EndDescr
+Wire Wire Line
+	6950 4250 7200 4250
 Connection ~ 8400 3550
 Wire Wire Line
@@
 Wire Wire Line
 	1900 2250 2000 2250
+Wire Wire Line
+	4600 2250 4600 2150
+$Comp
+L GND #PWR01
+U 1 1 5066EDF0
+P 4600 2250
+F 0 "#PWR01" H 4600 2250 30  0001 C CNN
+F 1 "GND" H 4600 2180 30  0001 C CNN
+	1    4600 2250
+	1    0    0    -1
+$EndComp
+Text Label 4000 2150 1    60   ~ 0
+BUSRESET
+$Comp
+L SW_PUSH SW4
+U 1 1 5066EDE6
+P 4300 2150
+F 0 "SW4" H 4450 2260 50  0000 C CNN
+F 1 "SW_PUSH" H 4300 2070 50  0000 C CNN
+	1    4300 2150
+	1    0    0    -1
+$EndComp
+$Comp
+L GND #PWR02
+U 1 1 5066ED17
+P 7700 4250
+F 0 "#PWR02" H 7700 4250 30  0001 C CNN
+F 1 "GND" H 7700 4180 30  0001 C CNN
+	1    7700 4250
+	0    -1   -1   0
+$EndComp
+$Comp
+L R R5
+U 1 1 5066ED0E
+P 7450 4250
+F 0 "R5" V 7530 4250 50  0000 C CNN
+F 1 "10KR" V 7450 4250 50  0000 C CNN
+	1    7450 4250
+	0    -1   -1   0
+$EndComp
+Text Label 7200 950  1    60   ~ 0
+BUSRESET
 $Comp
 L SWITCH_DSDP SW1
@@
 P 2450 2000
 F 0 "SW1" H 2450 2300 60  0000 C CNN
-F 1 "SWITCH_DSDP" H 2450 1650 60  0000 C CNN
+F 1 "WRITE" H 2450 1650 60  0000 C CNN
 	1    2450 2000
 	-1   0    0    1
@@
 MREQ
 $Comp
-L GND #PWR01
+L GND #PWR03
 U 1 1 5058E1E2
 P 1900 2250
-F 0 "#PWR01" H 1900 2250 30  0001 C CNN
+F 0 "#PWR03" H 1900 2250 30  0001 C CNN
 F 1 "GND" H 1900 2180 30  0001 C CNN
 	1    1900 2250
@@
 $EndComp
 $Comp
-L VCC #PWR02
+L VCC #PWR04
 U 1 1 5058E1DA
 P 1900 2050
-F 0 "#PWR02" H 1900 2150 30  0001 C CNN
+F 0 "#PWR04" H 1900 2150 30  0001 C CNN
 F 1 "VCC" H 1900 2150 30  0000 C CNN
 	1    1900 2050
@@
 $EndComp
 $Comp
-L VCC #PWR03
+L VCC #PWR05
 U 1 1 5058E15E
 P 2500 2750
-F 0 "#PWR03" H 2500 2850 30  0001 C CNN
+F 0 "#PWR05" H 2500 2850 30  0001 C CNN
 F 1 "VCC" H 2500 2850 30  0000 C CNN
 	1    2500 2750
@@
 /WE
 $Comp
-L VCC #PWR04
+L VCC #PWR06
 U 1 1 5058E0FB
 P 3450 1250
-F 0 "#PWR04" H 3450 1350 30  0001 C CNN
+F 0 "#PWR06" H 3450 1350 30  0001 C CNN
 F 1 "VCC" H 3450 1350 30  0000 C CNN
 	1    3450 1250
@@
 R0EN
 $Comp
-L VCC #PWR05
+L VCC #PWR07
 U 1 1 5058E067
 P 5950 4150
-F 0 "#PWR05" H 5950 4250 30  0001 C CNN
+F 0 "#PWR07" H 5950 4250 30  0001 C CNN
 F 1 "VCC" H 5950 4250 30  0000 C CNN
 	1    5950 4150
@@
 AR Path="/5058E053" Ref="SW2"  Part="1"
 F 0 "SW2" H 3750 1300 50  0000 C CNN
-F 1 "SWITCH_INV" H 3800 1000 50  0000 C CNN
+F 1 "ROM7" H 3800 1000 50  0000 C CNN
 	1    3950 1150
 	-1   0    0    1
@@
 P 6450 4250
 F 0 "SW3" H 6250 4400 50  0000 C CNN
-F 1 "SWITCH_INV" H 6300 4100 50  0000 C CNN
+F 1 "ROM0" H 6300 4100 50  0000 C CNN
 	1    6450 4250
 	-1   0    0    1
@@
 Q0
 $Comp
-L VCC #PWR06
+L VCC #PWR08
 U 1 1 5058D352
 P 8400 3050
-F 0 "#PWR06" H 8400 3150 30  0001 C CNN
+F 0 "#PWR08" H 8400 3150 30  0001 C CNN
 F 1 "VCC" H 8400 3150 30  0000 C CNN
 	1    8400 3050
@@
 	-1   0    0    1
 $EndComp
-Entry Wire Line
-	6200 -250 6300 -150
 $Comp
 L 74LS574 U1
@@
 CE
 $Comp
-L VCC #PWR07
+L VCC #PWR09
 U 1 1 4DDEB8E8
 P 9300 2350
-F 0 "#PWR07" H 9300 2450 30  0001 C CNN
+F 0 "#PWR09" H 9300 2450 30  0001 C CNN
 F 1 "VCC" H 9300 2450 30  0000 C CNN
 	1    9300 2350
@@
 RD
 $Comp
-L GND #PWR08
+L GND #PWR010
 U 1 1 4DC04C38
 P 1550 2800
-F 0 "#PWR08" H 1550 2800 30  0001 C CNN
+F 0 "#PWR010" H 1550 2800 30  0001 C CNN
 F 1 "GND" H 1550 2730 30  0001 C CNN
 	1    1550 2800
@@
 $EndComp
 $Comp
-L GND #PWR09
+L GND #PWR011
 U 1 1 4DBD3AB8
 P 9000 4550
-F 0 "#PWR09" H 9000 4550 30  0001 C CNN
+F 0 "#PWR011" H 9000 4550 30  0001 C CNN
 F 1 "GND" H 9000 4480 30  0001 C CNN
 	1    9000 4550
@@
 $EndComp
 $Comp
-L VCC #PWR010
+L VCC #PWR012
 U 1 1 4DBD3AB1
 P 9000 3950
-F 0 "#PWR010" H 9000 4050 30  0001 C CNN
+F 0 "#PWR012" H 9000 4050 30  0001 C CNN
 F 1 "VCC" H 9000 4050 30  0000 C CNN
 	1    9000 3950
@@
 Text GLabel 6600 950  1    60   Output ~ 0
 MREQ
-NoConn ~ 7200 950
 NoConn ~ 7100 950
 NoConn ~ 7000 950
@@
 Q3
 $Comp
-L VCC #PWR011
+L VCC #PWR013
 U 1 1 4DBBEA82
 P 6600 2100
-F 0 "#PWR011" H 6600 2200 30  0001 C CNN
+F 0 "#PWR013" H 6600 2200 30  0001 C CNN
 F 1 "VCC" H 6600 2200 30  0000 C CNN
 	1    6600 2100
@@
 D0
 $Comp
-L GND #PWR012
+L GND #PWR014
 U 1 1 4DBBE106
 P 9300 2450
-F 0 "#PWR012" H 9300 2450 30  0001 C CNN
+F 0 "#PWR014" H 9300 2450 30  0001 C CNN
 F 1 "GND" H 9300 2380 30  0001 C CNN
 	1    9300 2450
@@
 WR
 $Comp
-L GND #PWR013
+L GND #PWR015
 U 1 1 4CA89326
 P 7800 2150
-F 0 "#PWR013" H 7800 2150 30  0001 C CNN
+F 0 "#PWR015" H 7800 2150 30  0001 C CNN
 F 1 "GND" H 7800 2080 30  0001 C CNN
 	1    7800 2150
@@
 $EndComp
 $Comp
-L GND #PWR014
+L GND #PWR016
 U 1 1 4CA88AFC
 P 900 5400
-F 0 "#PWR014" H 900 5400 30  0001 C CNN
+F 0 "#PWR016" H 900 5400 30  0001 C CNN
 F 1 "GND" H 900 5330 30  0001 C CNN
 	1    900  5400
