File: CPC stuff/gordon/ramcard.sch (KiCad schematic (older format))
At the start: 24 parts, among them P1 CONN_25X2, SW1 WRITE, SW2 ROM7, SW3 ROM0, SW4 SW_PUSH, U1 74LS574, U2 74LS32, U3 74LS32, U4 74LS02, U5 74LS20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

Commit message: Oops ! Missing chip enable connection to the flash chip. This actually made me spot some ways to clean up the routing, but the first batch of board will have a Little Blue Strap (tm) on them.
git-svn-id: svn://pulkomandy.tk/avrstuff@77 c6672c3c-f6b6-47f9-9001-1fd6b12fecbe
Connections:
- net labels removed: CE
Changed lines of the file:
@@
-EESchema Schematic File Version 2  date 06/10/2012 12:12:36
+EESchema Schematic File Version 2  date 17/11/2012 12:11:23
 LIBS:device
 LIBS:power
@@
 Sheet 1 1
 Title "Ramcard"
-Date "29 sep 2012"
+Date "17 nov 2012"
 Rev ""
 Comp "Ram7"
@@
 /CE
 Text Label 6950 3450 0    60   ~ 0
-CE
+/CE
 $Comp
 L VCC #PWR09

Commit message: swap write switch pins to match hardware... This version is confirmed working.
git-svn-id: svn://pulkomandy.tk/avrstuff@81 c6672c3c-f6b6-47f9-9001-1fd6b12fecbe
Connections:
- net labels removed: RD
- no-connect marks 17 -> 19
Changed lines of the file:
@@
-EESchema Schematic File Version 2  date 17/11/2012 12:11:23
+EESchema Schematic File Version 2  date 28/11/2012 19:25:03
 LIBS:device
 LIBS:power
@@
 Sheet 1 1
 Title "Ramcard"
-Date "17 nov 2012"
+Date "28 nov 2012"
 Rev ""
 Comp "Ram7"
@@
 $EndDescr
 Wire Wire Line
+	6500 1900 6500 2100
+Wire Wire Line
+	6300 1900 6300 2100
+Wire Wire Line
 	6950 4250 7200 4250
 Connection ~ 8400 3550
@@
 Wire Wire Line
 	6200 1100 6200 800
-Wire Wire Line
-	6500 1900 6500 2200
-Wire Wire Line
-	6400 1900 6400 2200
-Wire Wire Line
-	6300 1900 6300 2200
-Wire Bus Line
-	6200 2200 6500 2200
 Connection ~ 2650 5050
 Connection ~ 2650 4950
@@
 Wire Wire Line
 	7400 2100 7400 1900
-Wire Wire Line
-	6200 1900 6200 2200
 Wire Bus Line
 	6200 800  6500 800
@@
 Wire Wire Line
 	4600 2250 4600 2150
+Wire Wire Line
+	6200 1900 6200 2100
+Wire Wire Line
+	6400 1900 6400 2100
+NoConn ~ 5400 950
+NoConn ~ 6800 950
 $Comp
 L GND #PWR01
@@
 	0    1    1    0
 $EndComp
-Text Label 6800 950  1    60   ~ 0
-RD
 $Comp
 L GND #PWR010
@@
 Entry Wire Line
 	6200 800  6100 700
-Entry Wire Line
-	6500 2200 6400 2100
-Entry Wire Line
-	6400 2200 6300 2100
-Entry Wire Line
-	6300 2200 6200 2100
-Entry Wire Line
-	6200 2200 6100 2100
 Text Label 6200 2100 1    60   ~ 0
 D7

Commit message: Rework FlashGordon
- New IO decoding to remove limitations and simplify routing
- Use SMD components to make the board smaller and prettier
Parts:
- removed D11, D2: DIODE, symbol DIODE
- removed R2: 1KR, symbol R
- removed U3: 74LS32, symbol 74LS32
- removed U4: 74LS02, symbol 74LS02
- removed U5: 74LS20, symbol 74LS20
- added U3, U5: 74LS138, Package_SO:SOIC-16_3.9x9.9mm_P1.27mm, symbol 74xx:74LS138
- added U4: 74LS00, Package_SO:SOIC-14_3.9x8.7mm_P1.27mm, symbol 74xx:74LS00
- C2, C3, C4: footprint (none) -> Capacitor_SMD:C_1206_3216Metric_Pad1.42x1.75mm_HandSolder; symbol C -> ramcard-rescue:C
- C5: footprint (none) -> Capacitor_THT:CP_Radial_D5.0mm_P2.50mm; symbol CP1 -> ramcard-rescue:CP1
- D1: footprint (none) -> LED_THT:LED_D3.0mm; symbol LED -> ramcard-rescue:LED
- D13: footprint (none) -> Diode_THT:D_A-405_P7.62mm_Horizontal; symbol DIODE -> ramcard-rescue:DIODE
- P1: footprint (none) -> Connector_IDC:IDC-Header_2x25_P2.54mm_Vertical; symbol CONN_25X2 -> ramcard-rescue:CONN_25X2
- R1, R3, R4, R5: footprint (none) -> Resistor_SMD:R_0805_2012Metric; symbol R -> ramcard-rescue:R
- SW1: footprint (none) -> Button_Switch_THT:SW_E-Switch_EG1271_DPDT; symbol SWITCH_DSDP -> byteeeprom:Switch_DSDP
- SW2, SW3: footprint (none) -> Connector_PinHeader_2.54mm:PinHeader_1x03_P2.54mm_Vertical; symbol SWITCH_INV -> ramcard-rescue:SWITCH_INV
- SW4: footprint (none) -> Button_Switch_SMD:SW_SPST_B3S-1000; symbol SW_PUSH -> ramcard-rescue:SW_PUSH
- U1: footprint (none) -> Package_SO:SOIC-20W_7.5x12.8mm_P1.27mm; symbol 74LS574 -> ramcard-rescue:74LS574
- U2: footprint (none) -> Package_SO:SOIC-14_3.9x8.7mm_P1.27mm; symbol 74LS32 -> ramcard-rescue:74LS32
- U6: footprint (none) -> Package_LCC:PLCC-32_11.4x14.0mm_P1.27mm; symbol 29C040 -> byteeeprom:29C040
Connections:
- net labels added: A14A15
- wire segments 134 -> 150
- no-connect marks 19 -> 30
Other:
- note added: "Disable switches"
- note added: "ROM address space decoding"
- note added: "Use Q7 instead for ROMs 32-63."
- note added: "Write protect switch"
- note removed: "comparator"
- moved on the sheet: C2, C3, C4, C5, D1, R1, R3, R5, SW2, SW3, SW4, U2A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

Commit message: Cleanups and improvements.
Parts:
- removed SW2: ROM7, Connector_PinHeader_2.54mm:PinHeader_1x03_P2.54mm_Vertical, symbol ramcard-rescue:SWITCH_INV
- removed SW3: ROM0, Connector_PinHeader_2.54mm:PinHeader_1x03_P2.54mm_Vertical, symbol ramcard-rescue:SWITCH_INV
- added JP1, JP2: Jumper_3_Open, Connector_PinHeader_2.54mm:PinHeader_1x03_P2.54mm_Vertical, symbol Jumper:Jumper_3_Open
- added JP3: Jumper_NC_Small, Jumper:SolderJumper-2_P1.3mm_Bridged_RoundedPad1.0x1.5mm, symbol Device:Jumper_NC_Small
- added JP4: Jumper_NO_Small, Jumper:SolderJumper-2_P1.3mm_Open_RoundedPad1.0x1.5mm, symbol Device:Jumper_NO_Small
- added unit 3 of U4
Connections:
- wire segments 150 -> 164
Other:
- note added: "All ROMs disabled \nwhen jumper unplugged"
- note added: "Power distribution"
- note added: "ROM activation decoding"
- note added: "ROM address space access (C000-FFFF) decoding"
- note added: "Reset button"
- note added: "Unused gate"
- note added: "Use Q7 for ROMs 32-63."
- note removed: "ROM address space decoding"
- note removed: "Rom active notification"
- note removed: "Use Q7 instead for ROMs 32-63."
- moved on the sheet: C2, C3, C4, C5, D13, R4, R5, SW4, U2A, U3, U4E, U5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

Commit message: Gordon: fix some problems in schematics
- Swapped pins on write switch
- Old symbols used for LED and Diode, the pins have been swapped in
  newer versions leading to mismatch between silkscreen and symbol
Parts:
- D1: symbol ramcard-rescue:LED -> Device:LED
- D13: symbol ramcard-rescue:DIODE -> Device:D
Other:
- moved on the sheet: D13
Changed lines of the file:
@@
 	1050 4350 900  4350
-Wire Wire Line
-	8900 3950 9050 3950
 Wire Wire Line
 	7600 1100 7600 950
@@
 Wire Wire Line
 	7450 2650 7600 2650
-Wire Wire Line
-	2650 1750 2700 1750
 Wire Wire Line
 	1050 950  950  950
@@
 Text Label 2150 850  0    60   ~ 0
 RDWR
+Text GLabel 950  950  0    60   Output ~ 0
+ROMEN
 Text GLabel 1150 750  0    60   Output ~ 0
-ROMEN
-Text GLabel 950  950  0    60   Output ~ 0
 MREQ
 $Comp
@@
 $EndComp
 $Comp
-L ramcard-rescue:LED D1
+L Device:LED D1
 U 1 1 5058E14C
-P 2450 1750
-F 0 "D1" H 2450 1850 50  0000 C CNN
-F 1 "LED" H 2450 1650 50  0000 C CNN
-F 2 "LED_THT:LED_D3.0mm" H 2450 1750 50  0001 C CNN
-F 3 "" H 2450 1750 50  0001 C CNN
-	1    2450 1750
-	1    0    0    -1
+P 2400 1750
+F 0 "D1" H 2400 1850 50  0000 C CNN
+F 1 "LED" H 2400 1650 50  0000 C CNN
+F 2 "LED_THT:LED_D3.0mm" H 2400 1750 50  0001 C CNN
+F 3 "" H 2400 1750 50  0001 C CNN
+	1    2400 1750
+	-1   0    0    1
 $EndComp
 $Comp
@@
 $EndComp
 $Comp
-L ramcard-rescue:DIODE D13
+L Device:D D13
 U 1 1 4CA870AA
-P 8700 3950
-F 0 "D13" H 8700 4050 40  0000 C CNN
-F 1 "DIODE" H 8700 3850 40  0000 C CNN
-F 2 "Diode_THT:D_A-405_P7.62mm_Horizontal" H 8700 3950 50  0001 C CNN
-F 3 "" H 8700 3950 50  0001 C CNN
-	1    8700 3950
-	1    0    0    -1
+P 8650 3950
+F 0 "D13" H 8650 4050 40  0000 C CNN
+F 1 "DIODE" H 8650 3850 40  0000 C CNN
+F 2 "Diode_THT:D_A-405_P7.62mm_Horizontal" H 8650 3950 50  0001 C CNN
+F 3 "" H 8650 3950 50  0001 C CNN
+	1    8650 3950
+	-1   0    0    1
 $EndComp
 Wire Wire Line
@@
 Wire Wire Line
 	4450 1500 3950 1500
+Wire Wire Line
+	2550 1750 2700 1750
+Wire Wire Line
+	8800 3950 9050 3950
 Wire Bus Line
 	6200 800  6500 800
