File: CPC stuff/gordon/ramcard.kicad_pcb (KiCad board)
At the start: 2 copper layers, 66 x 41.3 mm, 21 parts, among them P1 CONN_25X2, SW1 WRITE, SW2 ROM7, SW3 ROM0, SW4 SW_PUSH, U1 74LS574, U2 74LS32, U3 74LS138, U4 74LS00, U5 74LS138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

Commit message: Cleanups and improvements.
Parts:
- removed SW2: ROM7, Connector_PinHeader_2.54mm:PinHeader_1x03_P2.54mm_Vertical
- removed SW3: ROM0, Connector_PinHeader_2.54mm:PinHeader_1x03_P2.54mm_Vertical
- added JP1: Jumper_3_Open, Connector_PinHeader_2.54mm:PinHeader_1x03_P2.54mm_Vertical, F.Cu at (105.2, 33.8)
- added JP2: Jumper_3_Open, Connector_PinHeader_2.54mm:PinHeader_1x03_P2.54mm_Vertical, F.Cu at (108.5, 33.8)
- added JP3: Jumper_NC_Small, Jumper:SolderJumper-2_P1.3mm_Bridged_RoundedPad1.0x1.5mm, F.Cu at (90.7, 36.8)
- added JP4: Jumper_NO_Small, Jumper:SolderJumper-2_P1.3mm_Open_RoundedPad1.0x1.5mm, F.Cu at (90.7, 34.5)
- moved D13 24.8 mm to (105.3, 38.2)
- moved R4 24.8 mm to (105.3, 42.3)
- moved U1 24.8 mm to (85.3, 50.3)
- moved U2 24.8 mm to (87.0, 37.0)
- moved C5 24.8 mm to (52.6, 52.2)
- moved P1 24.8 mm to (48.1, 64.3)
- moved C2 24.8 mm to (54.5, 44.6)
- moved C4 24.8 mm to (86.9, 30.0)
- moved R1 24.8 mm to (71.0, 42.0)
- moved R3 24.8 mm to (79.9, 35.7)
- moved SW1 24.8 mm to (72.9, 39.5)
- moved U4 24.8 mm to (53.4, 37.1)
- moved U6 24.8 mm to (64.6, 50.9)
- moved C3 24.8 mm to (97.9, 30.0)
- moved D1 24.8 mm to (69.1, 39.5)
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Connections:
- U4 pad 10: //CE -> GND
- U4 pad 11: (no net) -> Net-(D13-Pad1)
- U4 pad 12: (no net) -> //CE
- U4 pad 13: (no net) -> //CE
- U4 pad 8: Net-(D13-Pad1) -> (no net)
- U4 pad 9: //CE -> GND
- U5 pad 12: /ROMACC -> Net-(JP3-Pad1)
- U5 pad 7: (no net) -> Net-(JP4-Pad1)
Routing:
- net GND: track 353.3 -> 294.0 mm, vias 3 -> 6
- net /ROMACC: track 21.8 -> 11.4 mm, vias 2 -> 1
- net VCC: track 189.5 -> 198.7 mm, vias 6 -> 5
- net Net-(JP3-Pad1): track 0.00 -> 9.09 mm, vias 0 -> 1
- net /A14A15: track 47.0 -> 52.6 mm, vias 2 -> 0
- net //CE: track 60.0 -> 55.7 mm
- net Net-(JP4-Pad1): track 0.00 -> 3.69 mm, vias 0 -> 1
- net Net-(JP2-Pad1): track 28.4 -> 24.9 mm
- net /A13: track 61.2 -> 58.6 mm
- net Net-(D13-Pad1): track 54.6 -> 56.2 mm
- net /Q1: track 60.1 -> 59.5 mm
Other:
- board text added: "0-31"
- board text added: "32-63"
- board text added: "OFF"
- board text added: "ON"
- board text added: "ROM0"
- board text added: "ROM7"
- board text removed: "ROM7 ROM0"

Commit message: Gordon: fix some problems in schematics
- Swapped pins on write switch
- Old symbols used for LED and Diode, the pins have been swapped in
  newer versions leading to mismatch between silkscreen and symbol
Parts:
- moved D13 7.75 mm to (105.3, 46.0), turned to 90 degrees
- moved D1 2.29 mm to (69.1, 37.2), turned to 270 degrees
- renumbered R5 to 10K, R1 to 1K, R4 to 1K, R3 to 220
Connections:
- 1K pad 2: Net-(D1-Pad1) -> Net-(D1-Pad2)
- 1K pad 1: Net-(D13-Pad1) -> Net-(D13-Pad2)
- 220 pad 1: Net-(D1-Pad2) -> Net-(D1-Pad1)
- D13 pad 1: Net-(D13-Pad1) -> ROMDIS
- D13 pad 2: ROMDIS -> Net-(D13-Pad2)
- SW1 pad 2: Net-(D1-Pad2) -> Net-(D1-Pad1)
- SW1 pad 4: MREQ -> ROMEN
- SW1 pad 6: ROMEN -> MREQ
- U4 pad 11: Net-(D13-Pad1) -> Net-(D13-Pad2)
Routing:
- net Net-(D13-Pad2): track 0.00 -> 56.2 mm, vias 0 -> 1
- net Net-(D13-Pad1): track 56.2 -> 0.00 mm, vias 1 -> 0
- net ROMEN: track 72.0 -> 50.7 mm
- net Net-(D1-Pad1): track 2.80 -> 14.0 mm
- net Net-(D1-Pad2): track 10.4 -> 2.80 mm
- net MREQ: track 31.0 -> 34.4 mm, vias 0 -> 1
- net /A13: track 58.6 -> 61.2 mm
- net //CE: track 55.7 -> 53.6 mm
- net VCC: track 198.7 -> 200.1 mm
Other:
- board text added: "HCT00"
- board text added: "HCT32"
