File: CPC stuff/dreamsound/dreamsound/dreamsound.sch (KiCad schematic (older format))
At the start: 13 parts, among them J1 Conn_02x25_Odd_Even, J2 Conn_02x07_Odd_Even, J3 DB25_Female, U1 74LS30, U2 74LS138, U3 74LS32

Commit message: Cleanups and improvements.
Parts:
- J3: footprint Connector_Dsub:DSUB-25_Female_Horizontal_P2.77x2.54mm_EdgePinOffset9.40mm -> Connector_Dsub:DSUB-25_Female_Horizontal_P2.77x2.84mm_EdgePinOffset4.94mm_Housed_MountingHolesOffset7.48mm
- U2: footprint Package_SO:SOIC-16_4.55x10.3mm_P1.27mm -> Package_SO:SOIC-16_3.9x9.9mm_P1.27mm
Connections:
- net A10: now also U1.1; no longer U1.3
- net A11: now also U1.2; no longer U1.4
- net A12: now also U1.3; no longer U1.5
- net A13: now also U1.4; no longer U1.6
- net A14: now also U1.5; no longer U1.12
- net A15: now also U1.6; no longer U1.11
- net A7: now also U1.12; no longer U1.1
- net A9: now also U1.11; no longer U1.2
- net !RESET: now reaches J1.41 (Pin_41)
- net !RESET: now also J3.10
- net !BUSRESET: no longer names the net of J1.40 (Pin_40)
- net !BUSRESET: no longer J3.10
Changed lines of the file:
@@
 EESchema Schematic File Version 4
+LIBS:dreamsound-cache
 EELAYER 26 0
 EELAYER END
@@
 F 0 "U2" H 2950 3078 50  0000 C CNN
 F 1 "74LS138" H 2950 2987 50  0000 C CNN
-F 2 "Package_SO:SOIC-16_4.55x10.3mm_P1.27mm" H 2950 2300 50  0001 C CNN
+F 2 "Package_SO:SOIC-16_3.9x9.9mm_P1.27mm" H 2950 2300 50  0001 C CNN
 F 3 "http://www.ti.com/lit/gpn/sn74LS138" H 2950 2300 50  0001 C CNN
 	1    2950 2300
@@
 Wire Wire Line
 	1400 1650 1650 1650
-Text Label 1650 2750 0    50   ~ 0
-!BUSRESET
 Wire Wire Line
 	1400 1750 1650 1750
@@
 	1400 2350 1650 2350
 Wire Wire Line
-	1400 2750 1650 2750
-Wire Wire Line
 	900  2350 650  2350
 Wire Wire Line
@@
 Wire Wire Line
 	900  2050 650  2050
+Text Label 2250 1550 0    50   ~ 0
+A7
+Text Label 2250 1450 0    50   ~ 0
+A9
 Text Label 2250 850  0    50   ~ 0
-A7
+A10
 Text Label 2250 950  0    50   ~ 0
-A9
+A11
 Text Label 2250 1050 0    50   ~ 0
-A10
+A12
 Text Label 2250 1150 0    50   ~ 0
-A11
+A13
 Text Label 2250 1250 0    50   ~ 0
-A12
+A14
 Text Label 2250 1350 0    50   ~ 0
-A13
-Text Label 2250 1550 0    50   ~ 0
-A14
-Text Label 2250 1450 0    50   ~ 0
 A15
-Text Label 2300 3050 0    50   ~ 0
-A1
 Text Label 2300 2500 0    50   ~ 0
 A2
@@
 F 0 "J3" H 10529 2196 50  0000 L CNN
 F 1 "DB25_Female" H 10529 2105 50  0000 L CNN
-F 2 "Connector_Dsub:DSUB-25_Female_Horizontal_P2.77x2.54mm_EdgePinOffset9.40mm" H 10350 2150 50  0001 C CNN
+F 2 "Connector_Dsub:DSUB-25_Female_Horizontal_P2.77x2.84mm_EdgePinOffset4.94mm_Housed_MountingHolesOffset7.48mm" H 10350 2150 50  0001 C CNN
 F 3 " ~" H 10350 2150 50  0001 C CNN
 	1    10350 2150
@@
 A0
 Text Label 9550 2750 0    50   ~ 0
-!BUSRESET
+!RESET
 Wire Wire Line
 	9800 950  10050 950
@@
 NoConn ~ 900  2650
 NoConn ~ 900  2750
-NoConn ~ 900  2850
+NoConn ~ 1400 2750
 NoConn ~ 900  2950
 NoConn ~ 900  3050
@@
 	9750 2050 9750 2250
 $Comp
-L power:GND #PWR?
+L power:GND #PWR0101
 U 1 1 5EAB0C0A
 P 9750 3350
-F 0 "#PWR?" H 9750 3100 50  0001 C CNN
+F 0 "#PWR0101" H 9750 3100 50  0001 C CNN
 F 1 "GND" H 9755 3177 50  0000 C CNN
 F 2 "" H 9750 3350 50  0001 C CNN
@@
 Connection ~ 9750 3250
 $Comp
-L power:VCC #PWR?
+L power:VCC #PWR0102
 U 1 1 5EAB5D51
 P 10050 3550
-F 0 "#PWR?" H 10050 3400 50  0001 C CNN
+F 0 "#PWR0102" H 10050 3400 50  0001 C CNN
 F 1 "VCC" H 10068 3723 50  0000 C CNN
 F 2 "" H 10050 3550 50  0001 C CNN
@@
 Wire Wire Line
 	10050 3550 10050 3350
+Wire Wire Line
+	900  2850 650  2850
+Text Label 650  2850 0    50   ~ 0
+!RESET
 $EndSCHEMATC

Commit message: Latest version of DreamSound/Willy and FlashGordon + Add Nova
Parts:
- removed JP1, JP2: Jumper_3_Open, Connector_PinHeader_2.54mm:PinHeader_1x03_P2.54mm_Vertical, symbol Jumper:Jumper_3_Open
- U3: footprint Package_SO:SOIC-14_3.9x8.7mm_P1.27mm -> (none)
Connections:
- net !RDCS is gone; now on net CSA1: U3.11
- net !RD: no longer U3.13
- net !WRCS: now also J3.16 (P16)
- net A1: now also U3.13
- net CSA1: now reaches J3.14 (P14)
Other:
- moved on the sheet: C1, C2, C3, C4, J3, JP3, U1B, U3C, U3E
